Commit message: first basic changes in the files for ec612

File: elite_description/urdf/elite_description.urdf.xacro (robot description, xacro)
@@ -5,8 +5,8 @@
 -->
 <robot xmlns:xacro="http://www.ros.org/wiki/xacro" name="elite">
-<!-- This is the main URDF file for ec66 elite arm-->
+<!-- This is the main URDF file for ec612 elite arm-->
   <!-- Set use_gz = true for Modern Gazebo Simulation-->
   <xacro:arg name="use_gz" default="false"/>
-  <xacro:arg name="arm_type" default="ec66"/>
+  <xacro:arg name="arm_type" default="ec612"/>
   <!-- Include macros -->
   <xacro:include filename="$(find elite_description)/urdf/xacros/elite_macro.xacro" />

File: elite_description/urdf/xacros/elite_macro.xacro (robot description, xacro)
@@ -45,5 +45,5 @@
       <visual>
       <geometry>
-        <mesh filename="package://elite_description/meshes/ec66/base_link.stl"/>
+        <mesh filename="package://elite_description/meshes/ec612/base_link.stl"/>
       </geometry>
       <material name="">
@@ -53,5 +53,5 @@
       <collision>
       <geometry>
-        <mesh filename="package://elite_description/meshes/ec66/base_link.stl"/>
+        <mesh filename="package://elite_description/meshes/ec612/base_link.stl"/>
       </geometry>
       </collision>
@@ -73,13 +73,13 @@
       <visual>
         <geometry>
-          <mesh filename="package://elite_description/meshes/ec66/link1.stl"/>
-        </geometry>
-        <material name="">
-          <color rgba="1 1 1 1" />
-        </material>
-      </visual>
-      <collision>
-        <geometry>
-          <mesh filename="package://elite_description/meshes/ec66/link1.stl"/>
+          <mesh filename="package://elite_description/meshes/ec612/link1.stl"/>
+        </geometry>
+        <material name="">
+          <color rgba="1 1 1 1" />
+        </material>
+      </visual>
+      <collision>
+        <geometry>
+          <mesh filename="package://elite_description/meshes/ec612/link1.stl"/>
         </geometry>
       </collision>
@@ -114,13 +114,13 @@
       <visual>
         <geometry>
-          <mesh filename="package://elite_description/meshes/ec66/link2.stl"/>
-        </geometry>
-        <material name="">
-          <color rgba="1 1 1 1" />
-        </material>
-      </visual>
-      <collision>
-        <geometry>
-          <mesh filename="package://elite_description/meshes/ec66/link2.stl"/>
+          <mesh filename="package://elite_description/meshes/ec612/link2.stl"/>
+        </geometry>
+        <material name="">
+          <color rgba="1 1 1 1" />
+        </material>
+      </visual>
+      <collision>
+        <geometry>
+          <mesh filename="package://elite_description/meshes/ec612/link2.stl"/>
         </geometry>
       </collision>
@@ -155,13 +155,13 @@
       <visual>
         <geometry>
-          <mesh filename="package://elite_description/meshes/ec66/link3.stl"/>
-        </geometry>
-        <material name="">
-          <color rgba="1 1 1 1" />
-        </material>
-      </visual>
-      <collision>
-        <geometry>
-          <mesh filename="package://elite_description/meshes/ec66/link3.stl"/>
+          <mesh filename="package://elite_description/meshes/ec612/link3.stl"/>
+        </geometry>
+        <material name="">
+          <color rgba="1 1 1 1" />
+        </material>
+      </visual>
+      <collision>
+        <geometry>
+          <mesh filename="package://elite_description/meshes/ec612/link3.stl"/>
         </geometry>
       </collision>
@@ -196,13 +196,13 @@
       <visual>
         <geometry>
-          <mesh filename="package://elite_description/meshes/ec66/link4.stl"/>
-        </geometry>
-        <material name="">
-          <color rgba="1 1 1 1" />
-        </material>
-      </visual>
-      <collision>
-        <geometry>
-          <mesh filename="package://elite_description/meshes/ec66/link4.stl"/>
+          <mesh filename="package://elite_description/meshes/ec612/link4.stl"/>
+        </geometry>
+        <material name="">
+          <color rgba="1 1 1 1" />
+        </material>
+      </visual>
+      <collision>
+        <geometry>
+          <mesh filename="package://elite_description/meshes/ec612/link4.stl"/>
         </geometry>
       </collision>
@@ -237,13 +237,13 @@
       <visual>
         <geometry>
-          <mesh filename="package://elite_description/meshes/ec66/link5.stl"/>
-        </geometry>
-        <material name="">
-          <color rgba="1 1 1 1" />
-        </material>
-      </visual>
-      <collision>
-        <geometry>
-          <mesh filename="package://elite_description/meshes/ec66/link5.stl"/>
+          <mesh filename="package://elite_description/meshes/ec612/link5.stl"/>
+        </geometry>
+        <material name="">
+          <color rgba="1 1 1 1" />
+        </material>
+      </visual>
+      <collision>
+        <geometry>
+          <mesh filename="package://elite_description/meshes/ec612/link5.stl"/>
         </geometry>
       </collision>
@@ -278,13 +278,13 @@
       <visual>
         <geometry>
-          <mesh filename="package://elite_description/meshes/ec66/link6.stl"/>
-        </geometry>
-        <material name="">
-          <color rgba="1 1 1 1" />
-        </material>
-      </visual>
-      <collision>
-        <geometry>
-          <mesh filename="package://elite_description/meshes/ec66/link6.stl"/>
+          <mesh filename="package://elite_description/meshes/ec612/link6.stl"/>
+        </geometry>
+        <material name="">
+          <color rgba="1 1 1 1" />
+        </material>
+      </visual>
+      <collision>
+        <geometry>
+          <mesh filename="package://elite_description/meshes/ec612/link6.stl"/>
         </geometry>
       </collision>

File: elite_moveit/config/ec612_simulation.urdf.xacro (robot description, xacro)
@@ -3,5 +3,5 @@
     <xacro:arg name="initial_positions_file" default="initial_positions.yaml" />
     <xacro:arg name="use_gz" default="true"/>
-    <xacro:arg name="arm_type" default="ec66"/>
+    <xacro:arg name="arm_type" default="ec612"/>
     <!-- Import ec612 urdf file with use_gaz set to true and arm argument-->
     <xacro:include filename="$(find elite_description)/urdf/elite_description.urdf.xacro"/>
